Commit message: Imported upstream version '1.0.0' of 'upstream'

File: dbw_fca_description/urdf/pacifica.urdf.xacro (robot description, xacro)
@@ -1,140 +1,4 @@
 <?xml version="1.0"?>
 <robot name="pacifica" xmlns:xacro="http://www.ros.org/wiki/xacro" >
-  <xacro:property name="half_track_width" value="0.77" />
-  <xacro:property name="half_wheelbase" value="1.54" />
-  <xacro:property name="wheel_radius" value="0.365" />
-  <xacro:property name="wheel_thickness" value="0.25" />
-  <xacro:property name="wheel_mass" value="10.0" />
-  <xacro:property name="body_mass" value="2242.0" />
-  <xacro:property name="body_width" value="${2*half_track_width}" />
-  <xacro:property name="body_depth" value="${2*half_wheelbase + 1.2}" />
-  <xacro:property name="body_length" value="0.6" />
-  <xacro:macro name="rear_wheel" params="name x y z flip" >
-    <link name="wheel_${name}" >
-      <visual>
-        <origin xyz="0 0 0" rpy="1.57079632679 ${flip * 3.1415926535} 0" />
-        <geometry>
-          <mesh filename="package://dbw_fca_description/meshes/wheel.dae" />
-        </geometry>
-      </visual>
-      <collision>
-        <geometry>
-          <cylinder radius="${wheel_radius}" length="${wheel_thickness}" />
-        </geometry>
-      </collision>
-      <inertial>
-        <origin xyz="0 0 0" rpy="0 0 0"/>
-        <mass value="${wheel_mass}"/>
-        <inertia ixx="${wheel_mass/12*(3*wheel_radius*wheel_radius + wheel_thickness*wheel_thickness)}" ixy="0" ixz="0" iyy="${wheel_mass/12*(3*wheel_radius*wheel_radius + wheel_thickness*wheel_thickness)}" iyz="0" izz="${wheel_mass/2 * wheel_radius*wheel_radius}"/>
-      </inertial>
-    </link>
-    <joint name="wheel_${name}" type="continuous" >
-      <parent link="base_link" />
-      <child link="wheel_${name}" />
-      <origin xyz="${x} ${y} ${z}" rpy="-1.57079632679 0 0" />
-      <axis xyz="0 0 1" />
-      <limit effort="0" velocity="22.0" />
-    </joint>
-  </xacro:macro>
-  <xacro:macro name="front_wheel" params="name x y z flip" >
-    <link name="wheel_${name}" >
-      <visual>
-        <origin xyz="0 0 0" rpy="1.57079632679 ${flip * pi} 0" />
-        <geometry>
-          <mesh filename="package://dbw_fca_description/meshes/wheel.dae" />
-        </geometry>
-      </visual>
-      <collision>
-        <geometry>
-          <cylinder radius="${wheel_radius}" length="${wheel_thickness}" />
-        </geometry>
-      </collision>
-      <inertial>
-        <origin xyz="0 0 0" rpy="0 0 0"/>
-        <mass value="${wheel_mass}"/>
-        <inertia ixx="${wheel_mass/12*(3*wheel_radius*wheel_radius + wheel_thickness*wheel_thickness)}" ixy="0" ixz="0" iyy="${wheel_mass/12*(3*wheel_radius*wheel_radius + wheel_thickness*wheel_thickness)}" iyz="0" izz="${wheel_mass/2 * wheel_radius*wheel_radius}"/>
-      </inertial>
-    </link>
-    <link name="steer_${name}" >
-      <inertial>
-        <origin xyz="-0.013054 -0.0295 0" rpy="0 0 0"/>
-        <mass value="1.0"/>
-        <inertia ixx="0.037227" ixy="0" ixz="0" iyy="0.04" iyz="0" izz="0.06"/>
-      </inertial>
-    </link>
-    <joint name="steer_${name}" type="revolute" >
-      <parent link="base_link" />
-      <child link="steer_${name}" />
-      <origin xyz="${x} ${y} ${z}" rpy="0 0 0" />
-      <axis xyz="0 0 1" />
-      <limit upper="0.6" lower="-0.6" effort="0.0" velocity="0.0" />
-    </joint>
-    <joint name="wheel_${name}" type="continuous" >
-      <parent link="steer_${name}" />
-      <child link="wheel_${name}" />
-      <origin xyz="0 0 0" rpy="-1.57079632679 0 0" />
-      <axis xyz="0 0 1" />
-      <limit effort="0" velocity="22.0" />
-    </joint>
-  </xacro:macro>
-  <link name="base_footprint" />
-  <link name="base_link" >
-    <visual>
-      <origin xyz="-0.06 0 0.1" rpy="0 0 0" />
-      <geometry>
-        <mesh filename="package://dbw_fca_description/meshes/body.dae" scale="0.96 0.96 0.96" />
-      </geometry>
-    </visual>
-    <collision>
-      <origin xyz="-0.06 0 0.1" rpy="0 0 0" />
-      <geometry>
-        <mesh filename="package://dbw_fca_description/meshes/body_collision.stl" scale="0.96 0.96 0.96" />
-      </geometry>
-      </collision>
-    <inertial>
-      <origin xyz="-0.25 0 0.3" rpy="0 0 0"/>
-      <mass value="${body_mass}"/>
-      <inertia ixx="${body_mass/12 * (body_width*body_width + body_length*body_length)}" ixy="0" ixz="0" iyy="${body_mass/12 * (body_length*body_length + body_depth*body_depth)}" iyz="0" izz="${body_mass/12 * (body_width*body_width + body_depth*body_depth)}"/>
-    </inertial>
-  </link>
-  <link name="hood_logo" >
-    <visual>
-      <origin xyz="-0.06 0 0.102" rpy="0 0 0" />
-      <geometry>
-        <mesh filename="package://dbw_fca_description/meshes/hood_logo.dae" scale="0.96 0.96 0.96" />
-      </geometry>
-    </visual>
-  </link>
-  <link name="door_logo" >
-    <visual>
-      <origin xyz="-0.06 0 0.102" rpy="0 0 0" />
-      <geometry>
-        <mesh filename="package://dbw_fca_description/meshes/door_logo.dae" scale="0.965 0.965 0.965" />
-      </geometry>
-    </visual>
-  </link>
-  <joint name="base_link" type="fixed" >
-    <parent link="base_footprint" />
-    <child link="base_link" />
-    <origin xyz="${half_wheelbase} 0 ${wheel_radius}" rpy="0 0 0" />
-  </joint>
-  <joint name="hood_logo" type="fixed" >
-    <parent link="base_link" />
-    <child link="hood_logo" />
-    <origin xyz="0 0 0" rpy="0 0 0" />
-  </joint>
-  <joint name="door_logo" type="fixed" >
-    <parent link="base_link" />
-    <child link="door_logo" />
-    <origin xyz="0 0 0" rpy="0 0 0" />
-  </joint>
-  <xacro:rear_wheel name="rl" x="${-half_wheelbase}" y="${half_track_width}" z="0" flip="0" />
-  <xacro:rear_wheel name="rr" x="${-half_wheelbase}" y="${-half_track_width}" z="0" flip="1" />
-  <xacro:front_wheel name="fl" x="${half_wheelbase}" y="${half_track_width}" z="0" flip="0" />
-  <xacro:front_wheel name="fr" x="${half_wheelbase}" y="${-half_track_width}" z="0" flip="1" />
-  <gazebo reference="hood_logo" >
-    <visual>
-      <transparency>0.01</transparency>
-    </visual>
-  </gazebo>
+  <xacro:include filename="$(find dbw_fca_description)/urdf/pacifica_18_structure.urdf.xacro" />
 </robot>
