Commit message: Imported upstream version '1.2.0' of 'upstream'

File: dbw_fca_description/urdf/jeep_18_structure.urdf.xacro (robot description, xacro)
@@ -30,5 +30,5 @@
       </inertial>
     </link>
-    <joint name="wheel_${name}" type="continuous" >
+    <joint name="wheel_${name}_joint" type="continuous" >
       <parent link="base_link" />
       <child link="wheel_${name}" />
@@ -64,5 +64,5 @@
       </inertial>
     </link>
-    <joint name="steer_${name}" type="revolute" >
+    <joint name="steer_${name}_joint" type="revolute" >
       <parent link="base_link" />
       <child link="steer_${name}" />
@@ -71,5 +71,5 @@
       <limit upper="0.6" lower="-0.6" effort="0.0" velocity="0.0" />
     </joint>
-    <joint name="wheel_${name}" type="continuous" >
+    <joint name="wheel_${name}_joint" type="continuous" >
       <parent link="steer_${name}" />
       <child link="wheel_${name}" />
@@ -107,10 +107,10 @@
     </visual>
   </link>
-  <joint name="base_link" type="fixed" >
+  <joint name="base_link_joint" type="fixed" >
     <parent link="base_footprint" />
     <child link="base_link" />
     <origin xyz="${half_wheelbase} 0 ${wheel_radius}" rpy="0 0 0" />
   </joint>
-  <joint name="hood_logo" type="fixed" >
+  <joint name="hood_logo_joint" type="fixed" >
     <parent link="base_link" />
     <child link="hood_logo" />

File: dbw_fca_description/urdf/pacifica_18_structure.urdf.xacro (robot description, xacro)
@@ -30,5 +30,5 @@
       </inertial>
     </link>
-    <joint name="wheel_${name}" type="continuous" >
+    <joint name="wheel_${name}_joint" type="continuous" >
       <parent link="base_link" />
       <child link="wheel_${name}" />
@@ -64,5 +64,5 @@
       </inertial>
     </link>
-    <joint name="steer_${name}" type="revolute" >
+    <joint name="steer_${name}_joint" type="revolute" >
       <parent link="base_link" />
       <child link="steer_${name}" />
@@ -71,5 +71,5 @@
       <limit upper="0.6" lower="-0.6" effort="0.0" velocity="0.0" />
     </joint>
-    <joint name="wheel_${name}" type="continuous" >
+    <joint name="wheel_${name}_joint" type="continuous" >
       <parent link="steer_${name}" />
       <child link="wheel_${name}" />
@@ -115,15 +115,15 @@
     </visual>
   </link>
-  <joint name="base_link" type="fixed" >
+  <joint name="base_link_joint" type="fixed" >
     <parent link="base_footprint" />
     <child link="base_link" />
     <origin xyz="${half_wheelbase} 0 ${wheel_radius}" rpy="0 0 0" />
   </joint>
-  <joint name="hood_logo" type="fixed" >
+  <joint name="hood_logo_joint" type="fixed" >
     <parent link="base_link" />
     <child link="hood_logo" />
     <origin xyz="0 0 0" rpy="0 0 0" />
   </joint>
-  <joint name="door_logo" type="fixed" >
+  <joint name="door_logo_joint" type="fixed" >
     <parent link="base_link" />
     <child link="door_logo" />
